Commit message: Rename shared plugin xacro to quad_gazebo.xacro
The plugin block is shared by every airframe, not just the F450.

File: urdf/build03.urdf.xacro (robot description, xacro)
@@ -8,5 +8,5 @@
   <xacro:include filename="$(find my_drone)/urdf/quad_mesh_common.xacro"/>
   <xacro:include filename="$(find my_drone)/urdf/build03_params.xacro"/>
-  <xacro:include filename="$(find my_drone)/urdf/f450_gazebo.xacro"/>
+  <xacro:include filename="$(find my_drone)/urdf/quad_gazebo.xacro"/>
   <material name="frame_grey"><color rgba="0.22 0.22 0.25 1.0"/></material>
   <xacro:macro name="frame_part" params="file">
@@ -50,4 +50,4 @@
   </link>
   <xacro:quad_rotors/>
-  <xacro:f450_gazebo_plugins/>
+  <xacro:quad_gazebo_plugins/>
 </robot>

File: urdf/f450.urdf.xacro (robot description, xacro)
@@ -20,5 +20,5 @@
 <robot name="f450" xmlns:xacro="http://www.ros.org/wiki/xacro">
   <xacro:include filename="$(find my_drone)/urdf/f450_params.xacro"/>
-  <xacro:include filename="$(find my_drone)/urdf/f450_gazebo.xacro"/>
+  <xacro:include filename="$(find my_drone)/urdf/quad_gazebo.xacro"/>
   <material name="carbon">  <color rgba="0.15 0.15 0.17 1.0"/></material>
   <material name="red_arm"> <color rgba="0.80 0.10 0.10 1.0"/></material>
@@ -134,4 +134,4 @@
   <xacro:rotor number="3" x="${-rotor_xy}" y="${-rotor_xy}"/>  <!-- rear-right,  cw  -->
   <!-- ==================== PLUGINS ==================== -->
-  <xacro:f450_gazebo_plugins/>
+  <xacro:quad_gazebo_plugins/>
 </robot>

File: urdf/jeno7.urdf.xacro (robot description, xacro)
@@ -8,5 +8,5 @@
   <xacro:include filename="$(find my_drone)/urdf/quad_mesh_common.xacro"/>
   <xacro:include filename="$(find my_drone)/urdf/jeno7_params.xacro"/>
-  <xacro:include filename="$(find my_drone)/urdf/f450_gazebo.xacro"/>
+  <xacro:include filename="$(find my_drone)/urdf/quad_gazebo.xacro"/>
   <material name="frame_carbon"><color rgba="0.15 0.15 0.17 1.0"/></material>
   <link name="base_link">
@@ -33,4 +33,4 @@
   </link>
   <xacro:quad_rotors/>
-  <xacro:f450_gazebo_plugins/>
+  <xacro:quad_gazebo_plugins/>
 </robot>

File: urdf/quad_gazebo.xacro (robot description, xacro)
@@ -2,5 +2,5 @@
 <!--
   Gazebo Harmonic (gz-sim 8) plugin blocks, shared by every quad in this
-  package (f450, build03, jeno7). All numbers come from <drone>_params.xacro.
+  package. All numbers come from <drone>_params.xacro.
   Two layers are declared here:
     1. MulticopterMotorModel  x4 - turns a commanded rotor velocity into
@@ -46,5 +46,5 @@
     </rotor>
   </xacro:macro>
-  <xacro:macro name="f450_gazebo_plugins" params="">
+  <xacro:macro name="quad_gazebo_plugins" params="">
     <xacro:motor_plugin number="0" direction="ccw"/>
     <xacro:motor_plugin number="1" direction="ccw"/>

File: urdf/quad_mesh_common.xacro (robot description, xacro)
@@ -4,5 +4,5 @@
   7040 tri-blade props, both meshes in mm with their axis on the origin and
   their base at z=0.
-  Rotor numbering and spin match f450.urdf.xacro and f450_gazebo.xacro, and
+  Rotor numbering and spin match quad_gazebo.xacro, and
   the standard props-in layout seen from above:
         FL (2) CW      FR (0) CCW
