Commit message: Split into description, control, teleop and bringup packages
Header-only control lib, relative topics, range-checked parameters.

File: my_drone_description/urdf/build03.urdf.xacro (robot description, xacro)
@@ -6,7 +6,7 @@
 -->
 <robot name="build03" xmlns:xacro="http://www.ros.org/wiki/xacro">
-  <xacro:include filename="$(find my_drone)/urdf/quad_mesh_common.xacro"/>
-  <xacro:include filename="$(find my_drone)/urdf/build03_params.xacro"/>
-  <xacro:include filename="$(find my_drone)/urdf/quad_gazebo.xacro"/>
+  <xacro:include filename="$(find my_drone_description)/urdf/quad_mesh_common.xacro"/>
+  <xacro:include filename="$(find my_drone_description)/urdf/build03_params.xacro"/>
+  <xacro:include filename="$(find my_drone_description)/urdf/quad_gazebo.xacro"/>
   <material name="frame_grey"><color rgba="0.22 0.22 0.25 1.0"/></material>
   <xacro:macro name="frame_part" params="file">
@@ -14,5 +14,5 @@
       <origin xyz="${cad_offset}" rpy="0 0 0"/>
       <geometry>
-        <mesh filename="package://my_drone/meshes/build03/${file}.stl" scale="${mesh_scale}"/>
+        <mesh filename="package://my_drone_description/meshes/build03/${file}.stl" scale="${mesh_scale}"/>
       </geometry>
       <material name="frame_grey"/>

File: my_drone_description/urdf/quad_mesh_common.xacro (robot description, xacro)
@@ -56,5 +56,5 @@
       <visual>
         <geometry>
-          <mesh filename="package://my_drone/meshes/common/Prop_7040-3_${spin}.stl" scale="${mesh_scale}"/>
+          <mesh filename="package://my_drone_description/meshes/common/Prop_7040-3_${spin}.stl" scale="${mesh_scale}"/>
         </geometry>
         <material name="prop_black"/>
@@ -63,5 +63,5 @@
         <origin xyz="0 0 ${prop_mesh_h}" rpy="0 0 0"/>
         <geometry>
-          <mesh filename="package://my_drone/meshes/common/Nut_M5_flange.stl" scale="${mesh_scale}"/>
+          <mesh filename="package://my_drone_description/meshes/common/Nut_M5_flange.stl" scale="${mesh_scale}"/>
         </geometry>
         <material name="nut_red"/>
@@ -84,5 +84,5 @@
       <origin xyz="${x} ${y} ${z}" rpy="0 0 0"/>
       <geometry>
-        <mesh filename="package://my_drone/meshes/common/Motor_2807SL.stl" scale="${mesh_scale}"/>
+        <mesh filename="package://my_drone_description/meshes/common/Motor_2807SL.stl" scale="${mesh_scale}"/>
       </geometry>
       <material name="motor_grey"/>
