Commit message: Fly PX4 through our topics; retire controller:=gz
my_drone_px4 holds the airframe and an offboard adapter; goto and teleop run unchanged on PX4.

File: my_drone_description/urdf/build03_params.xacro (robot description, xacro)
@@ -29,17 +29,4 @@
   <xacro:property name="rotor_z"       value=" 0.0174"/>   <!-- prop hub bottom -->
   <xacro:property name="motor_base_z"  value="-0.0093"/>
-  <!-- ==================== VELOCITY CONTROLLER ====================
-       gz divides attitude/rate gains by inertia and velocity gain by mass.
-       These are the proven F450 tune (git tag f450-final: 0.90 kg,
-       Ixx=Iyy=0.0098, Izz=0.0192; attitude 2.0 2.0 0.15, rate 0.4 0.4 0.18,
-       velocity 2.7) scaled by I_build03/I_f450 per axis (0.73, 0.77, 0.71)
-       and by mass (1.03), so the response matches. If you retune after
-       weighing, scale by the new inertia the same way. -->
-  <xacro:property name="velocity_gain"     value="2.79 2.79 2.79"/>
-  <xacro:property name="attitude_gain"     value="1.45 1.54 0.106"/>
-  <xacro:property name="angular_rate_gain" value="0.29 0.31 0.128"/>
-  <xacro:property name="max_linear_accel"  value="3 3 3"/>
-  <xacro:property name="max_linear_vel"    value="5 5 3"/>
-  <xacro:property name="max_angular_vel"   value="3 3 2"/>
   <xacro:property name="robot_ns" value="build03"/>
 </robot>

File: my_drone_description/urdf/quad_gazebo.xacro (robot description, xacro)
@@ -3,15 +3,10 @@
   Gazebo Harmonic (gz-sim 8) plugin blocks, shared by every quad in this
   package. All numbers come from <drone>_params.xacro.
-  Two layers are declared here:
-    1. MulticopterMotorModel  x4 - turns a commanded rotor velocity into
-       thrust and drag torque. This is the "ESC + motor + prop" model.
-    2. The controller that drives those four motors. With the xacro arg
-       controller:=custom (default) that is our flight_controller node,
-       which reads the <quad_physics> element below and publishes rotor
-       speeds. controller:=gz uses Gazebo's built-in
-       MulticopterVelocityControl instead (kept for A/B comparison).
+  MulticopterMotorModel x4 turns a commanded rotor velocity into thrust and
+  drag torque (the "ESC + motor + prop" model). The commands come from our
+  flight_controller (which reads the <quad_physics> element below) or from
+  PX4, on the same gz topic. Then the sensors and the exact-state odometry.
 -->
 <robot xmlns:xacro="http://www.ros.org/wiki/xacro">
-  <xacro:arg name="controller" default="custom"/>
   <!-- ============ Motor model, instantiated once per rotor ============ -->
   <xacro:macro name="motor_plugin" params="number direction">
@@ -37,14 +32,4 @@
     </gazebo>
   </xacro:macro>
-  <!-- direction 1 == ccw, -1 == cw, and must agree with turningDirection above.
-       Diagonally opposite rotors share a direction so yaw torque cancels. -->
-  <xacro:macro name="rotor_config_entry" params="number dir">
-    <rotor>
-      <jointName>rotor_${number}_joint</jointName>
-      <forceConstant>${motor_constant}</forceConstant>
-      <momentConstant>${moment_constant}</momentConstant>
-      <direction>${dir}</direction>
-    </rotor>
-  </xacro:macro>
   <xacro:macro name="quad_gazebo_plugins" params="">
     <xacro:motor_plugin number="0" direction="ccw"/>
@@ -67,33 +52,4 @@
       <rotor number="3" x="${rotor_x_rear}"  y="${-rotor_y}" direction="-1"/>
     </quad_physics>
-    <xacro:if value="${'$(arg controller)' == 'gz'}">
-    <!-- ============ Built-in velocity / attitude controller ============
-         Gains and limits come from <drone>_params.xacro. They are the
-         numbers most likely to need a tuning pass if the drone feels
-         sluggish (raise) or oscillates (lower).
-         Subscribes on:  /${robot_ns}/gazebo/command/twist
-         Enable on:      /${robot_ns}/enable                             -->
-    <gazebo>
-      <plugin filename="gz-sim-multicopter-control-system"
-              name="gz::sim::systems::MulticopterVelocityControl">
-        <robotNamespace>${robot_ns}</robotNamespace>
-        <commandSubTopic>gazebo/command/twist</commandSubTopic>
-        <enableSubTopic>enable</enableSubTopic>
-        <comLinkName>base_link</comLinkName>
-        <velocityGain>${velocity_gain}</velocityGain>
-        <attitudeGain>${attitude_gain}</attitudeGain>
-        <angularRateGain>${angular_rate_gain}</angularRateGain>
-        <maximumLinearAcceleration>${max_linear_accel}</maximumLinearAcceleration>
-        <maximumLinearVelocity>${max_linear_vel}</maximumLinearVelocity>
-        <maximumAngularVelocity>${max_angular_vel}</maximumAngularVelocity>
-        <rotorConfiguration>
-          <xacro:rotor_config_entry number="0" dir="1"/>
-          <xacro:rotor_config_entry number="1" dir="1"/>
-          <xacro:rotor_config_entry number="2" dir="-1"/>
-          <xacro:rotor_config_entry number="3" dir="-1"/>
-        </rotorConfiguration>
-      </plugin>
-    </gazebo>
-    </xacro:if>
     <!-- ============ Odometry: the exact state (ground truth) ============ -->
     <gazebo>
